Commit message: Update rect prism object

File: models/polygonal_prism/polygonal_prism.urdf (robot description, URDF)
Before this commit: robot box, 1 links, 0 joints
Links:
- link object_link: geometry collision mesh filename=package://grf_transport/models/polygonal_prism/polygonal_pr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 scale=1.0 1.0 1.0; visual mesh filename=package://grf_transport/models/polygonal_prism/polygonal_pr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 scale=1.0 1.0 1.0
