Commit message: Update objects friction

File: models/cylinder_prism/cylinder_prism_target.urdf (robot description, URDF)
Before this commit: robot target_box, 1 links, 0 joints
Links:
- link target_link: geometry visual mesh filename=package://grf_transport/models/cylinder_prism/cylinder_pris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 scale=1.0 1.0 0.05

File: models/l_shaped_prism/l_shaped_prism.urdf (robot description, URDF)
Before this commit: robot box, 1 links, 0 joints
Links:
- link object_link: geometry collision mesh filename=package://grf_transport/models/l_shaped_prism/l_shaped_pris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 scale=1.0 1.0 1.0; visual mesh filename=package://grf_transport/models/l_shaped_prism/l_shaped_pris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 scale=1.0 1.0 1.0

File: models/l_shaped_prism/l_shaped_prism_target.urdf (robot description, URDF)
Before this commit: robot target_box, 1 links, 0 joints
Links:
- link target_link: geometry visual mesh filename=package://grf_transport/models/l_shaped_prism/l_shaped_pris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 scale=1.0 1.0 0.05

File: models/polygonal_prism/polygonal_prism_target.urdf (robot description, URDF)
Before this commit: robot target_box, 1 links, 0 joints
Links:
- link target_link: geometry visual mesh filename=package://grf_transport/models/polygonal_prism/polygonal_pr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 scale=1.0 1.0 0.05

File: models/rectangular_prism/rectangular_prism.urdf (robot description, URDF)
Before this commit: robot box, 1 links, 0 joints
Links:
- link object_link: geometry collision mesh filename=package://grf_transport/models/rectangular_prism/rectangula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 scale=1.0 1.0 1.0; visual mesh filename=package://grf_transport/models/rectangular_prism/rectangula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 scale=1.0 1.0 1.0

File: models/rectangular_prism/rectangular_prism_target.urdf (robot description, URDF)
Before this commit: robot target_box, 1 links, 0 joints
Links:
- link target_link: geometry visual mesh filename=package://grf_transport/models/rectangular_prism/rectangula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 scale=1.0 1.0 0.05

File: models/triangular_prism/triangular_prism.urdf (robot description, URDF)
Before this commit: robot box, 1 links, 0 joints
Links:
- link object_link: geometry collision mesh filename=package://grf_transport/models/triangular_prism/triangular_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 scale=1.0 1.0 1.0; visual mesh filename=package://grf_transport/models/triangular_prism/triangular_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 scale=1.0 1.0 1.0

File: models/triangular_prism/triangular_prism_target.urdf (robot description, URDF)
Before this commit: robot target_box, 1 links, 0 joints
Links:
- link target_link: geometry visual mesh filename=package://grf_transport/models/triangular_prism/triangular_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 scale=1.0 1.0 0.05

File: models/u_shaped_prism/u_shaped_prism.urdf (robot description, URDF)
Before this commit: robot box, 1 links, 0 joints
Links:
- link object_link: geometry collision mesh filename=package://grf_transport/models/u_shaped_prism/u_shaped_pris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 scale=1.0 1.0 1.0; visual mesh filename=package://grf_transport/models/u_shaped_prism/u_shaped_pris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 scale=1.0 1.0 1.0

File: models/u_shaped_prism/u_shaped_prism_target.urdf (robot description, URDF)
Before this commit: robot target_box, 1 links, 0 joints
Links:
- link target_link: geometry visual mesh filename=package://grf_transport/models/u_shaped_prism/u_shaped_pris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 scale=1.0 1.0 0.05
